File: DIAGRAMAS DE FLUJO DE DISEÑO/wetLandCare/wetLandCare.kicad_pcb (KiCad board)
At the start: 2 copper layers, 105 x 75 mm, 36 parts, among them J1 M1ML1_CONTROL, J11 Barrel_Jack_MountingPin, J12 M2MR1_CONTROL, J2 Conn_01x01_Pin, J3 Screw_Terminal_01x03, J4 Conn_01x03_Socket, J5 Conn_01x03_Socket, J6 Conn_01x06_Socket, J7 M3RL1_BLOCK, J8 M4RR1_BLOCK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

Commit message: updated kicad files
Parts:
- removed J7: M3RL1_BLOCK, TerminalBlock:TerminalBlock_Altech_AK300-2_P5.00mm
- removed J8: M4RR1_BLOCK, TerminalBlock:TerminalBlock_Altech_AK300-2_P5.00mm
- added J9: Screw_Terminal_01x04, TerminalBlock:TerminalBlock_Altech_AK300-4_P5.00mm, F.Cu at (207.7, 98.3)
Connections:
- U5 pad 0: /PWM_MR -> /BAT_LVL_SENS
- U5 pad 5: /BAT_LVL_SENS -> /PWM_MR
Routing:
- net /5V_DRIVERS: track 155.0 -> 187.2 mm
- net VCC: track 196.5 -> 207.3 mm, vias 0 -> 1
- net Net-(J9-Pin_4): track 20.2 -> 30.9 mm
- net Net-(J12-Pin_2): track 103.4 -> 102.9 mm
- net Net-(U4-1A): track 104.2 -> 103.7 mm
- net GND: track 64.7 -> 64.8 mm, vias 14 -> 16
Other:
- board text added: "5V"
- board text added: "5V DRIVERS"
- board text added: "5V MCU"
- board text added: "DI1_3"
- board text added: "DI1_4"
- board text added: "DI2_3"
- board text added: "DI2_4"
- board text added: "ESP32-C3 SUPER MINI"
- board text added: "GND"
- board text added: "L298 SUPPLY"
- board text added: "MOTOR 3 LOGIC"
- board text added: "MOTOR 4 LOGIC"
- board text added: "MOTOR A"
- board text added: "MOTOR B"
- board text added: "PWM_3"
- board text added: "PWM_4"
- board text added: "VCC"
- board text added: "WetLandCare V2"
- board text removed: "WetLandCare v1.0"
